File: clap switch.kicad_pcb (KiCad board)
At the start: 2 copper layers, 14 parts, among them Q1 BC547, Q2 BC547, U1 NE555D

Commit message: updated clap switch project
Parts:
- removed BT1: Battery, Battery:BatteryHolder_Keystone_106_1x20mm
- added B1: 6V, Connector_PinHeader_2.54mm:PinHeader_1x02_P2.54mm_Vertical, F.Cu at (180.3, 80.8)
- added REF**: ., MountingHole:MountingHole_2.2mm_M2, F.Cu at (122.6, 95.6)
- added REF**: ., MountingHole:MountingHole_2.2mm_M2, F.Cu at (122.9, 70.7)
- added REF**: ., MountingHole:MountingHole_2.2mm_M2, F.Cu at (184.4, 70.6)
- added REF**: ., MountingHole:MountingHole_2.2mm_M2, F.Cu at (184.3, 95.9)
- C1: value C -> 100uF; footprint Capacitor_THT:C_Disc_D3.4mm_W2.1mm_P2.50mm -> Capacitor_THT:CP_Axial_L10.0mm_D4.5mm_P15.00mm_Horizontal
- C2: value C -> 0.1uF; footprint Capacitor_THT:C_Disc_D3.4mm_W2.1mm_P2.50mm -> Capacitor_THT:C_Disc_D5.0mm_W2.5mm_P2.50mm
- C3: value C_Polarized -> 0.1uF; footprint Capacitor_THT:CP_Radial_D4.0mm_P2.00mm -> Capacitor_THT:C_Disc_D5.0mm_W2.5mm_P2.50mm
- D1: footprint LED_THT:LED_D3.0mm -> LED_THT:LED_D5.0mm
- MK1: value Microphone_Condenser -> ~; footprint Connector_PinSocket_2.54mm:PinSocket_1x02_P2.54mm_Horizontal -> Connector_PinHeader_2.54mm:PinHeader_1x02_P2.54mm_Vertical
- R1: value R -> 4.7K
- R2: value R -> 1K
- R3: value R -> 470
- R4: value R -> 10K
- R5: value R -> 330
- U1: value NE555D -> NE555P
- moved C1 52.0 mm to (178.0, 91.7)
- moved MK1 27.9 mm to (128.2, 75.4), turned to 180 degrees
- moved D1 27.3 mm to (146.6, 91.4)
- moved R1 27.1 mm to (128.3, 80.8)
- moved U1 26.6 mm to (158.6, 77.2)
- moved R4 26.5 mm to (173.1, 77.3)
- moved R5 25.4 mm to (152.0, 79.2)
- moved R3 24.7 mm to (144.1, 71.6)
- moved R2 24.7 mm to (135.1, 71.7)
- moved Q1 24.5 mm to (135.0, 83.3)
- moved Q2 24.5 mm to (143.8, 83.5)
- moved C2 20.6 mm to (151.2, 75.6), turned to 0 degrees
- moved C3 8.68 mm to (155.4, 90.9), turned to 0 degrees
Connections:
- net +5V renamed Net-(B1-+)
- C1 pad 1: Net-(U1-CONT) -> Net-(U1-DISCH)
- C2 pad 1: Net-(U1-TRIG) -> Net-(Q2-C)
- C2 pad 2: Net-(Q2-C) -> Net-(U1-TRIG)
- C3 pad 1: Net-(U1-DISCH) -> GND
- C3 pad 2: GND -> Net-(U1-CONT)
Routing:
- net GND: track 190.3 -> 80.1 mm
- net Net-(B1-+): track 99.2 -> 69.6 mm
- net Net-(MK1--): track 42.7 -> 13.7 mm
- net Net-(U1-TRIG): track 0.00 -> 7.28 mm
- net Net-(Q2-C): track 8.57 -> 13.0 mm
- net Net-(U1-CONT): track 9.23 -> 12.3 mm
- net Net-(U1-OUT): track 5.08 -> 7.84 mm
- net Net-(U1-DISCH): track 20.1 -> 21.2 mm
Other:
- board outline added: 67.6 x 30.7 mm
- board text added: "Main Sheet"
